Commit message: test: Move object with rospy

File: team2_gazebo/urdf/camera.urdf.xacro (robot description, xacro)
@@ -2,9 +2,10 @@
 <robot name="camera" xmlns:xacro="http://www.ros.org/wiki/xacro">
   <xacro:property name="camera_link" value="0.05" />
-  <xacro:property name="ch" value="1.8" />
+  <xacro:property name="camera_height" value="2.0" />
+  <xacro:property name="camera_x" value="0.0" />
   <link name="world"/>
   <joint name="camera_joint" type="fixed">
     <axis xyz="0 1 0" />
-    <origin xyz="0 0 ${ch}" rpy="0 ${pi/2} 0"/>
+    <origin xyz="${camera_x} 0 ${camera_height}" rpy="0 ${pi/2} 0"/>
     <parent link="world"/>
     <child link="camera_link"/>

Commit message: test: Import fetch into camera world and clean up world models

File: team2_gazebo/urdf/camera.urdf.xacro (robot description, xacro)
@@ -2,5 +2,5 @@
 <robot name="camera" xmlns:xacro="http://www.ros.org/wiki/xacro">
   <xacro:property name="camera_link" value="0.05" />
-  <xacro:property name="camera_height" value="2.0" />
+  <xacro:property name="camera_height" value="0.0" />
   <xacro:property name="camera_x" value="0.0" />
   <link name="world"/>
